Commit message: 7.Robot Sensors

File: project2/src/my_robot/urdf/my_robot.xacro (robot description, xacro)
@@ -101,7 +101,6 @@
     </inertial>
   </link>
-  <!--
   <link name="camera">
-    <pose> 0 0 0 0 0 0 </pose>
+    <!-- <pose> 0 0 0 0 0 0 </pose> -->
     <visual name='camera_visual'>
       <origin xyz="0 0 0" rpy="0 0 0"/>
@@ -109,4 +108,11 @@
         <box size=".05 .05 .05"/>
       </geometry>
+    </visual>
+    <collision name='camera_collision'>
+      <origin xyz="0 0 0" rpy="0 0 0"/>
+      <geometry>
+        <box size=".05 .05 .05"/>
+      </geometry>
+    </collision>
     <inertial>
       <mass value="0.1"/>
@@ -118,5 +124,27 @@
     </inertial>
   </link>
-  -->
+  <link name="hokuyo">
+    <!-- <pose> 0 0 0 0 0 0 </pose> -->
+    <visual name='hokuyo_visual'>
+      <origin xyz="0 0 0" rpy="0 0 0"/>
+      <geometry>
+        <mesh filename="package://my_robot/meshes/hokuyo.dae"/>
+      </geometry>
+      <material name="black"/>
+    </visual>
+    <collision name='hokuyo_collision'>
+      <geometry>
+        <box size="0.1 0.1 0.1"/>
+      </geometry>
+    </collision>
+    <inertial>
+      <mass value="1e-5"/>
+      <inertia
+        ixx="1e-6" ixy="0" ixz="0"
+        iyy="1e-6" iyz="0"
+        izz="1e-6"
+      />
+    </inertial>
+  </link>
   <joint type="continuous" name="left_wheel_hinge">
     <origin xyz="-0.15 0.15 0" rpy="0 0 0"/>
@@ -135,3 +163,15 @@
     <dynamics damping="1.0" friction="1.0"/>
   </joint>
+  <joint type="fixed" name="camera_joint">
+    <origin xyz="0.2 0 0" rpy="0 0 0"/>
+    <child link="camera"/>
+    <parent link="chassis"/>
+    <axis xyz="0 1 0" rpy="0 0 0"/>
+  </joint>
+  <joint type="fixed" name="hokuyo_joint">
+    <origin xyz="0.15 0 0.1" rpy="0 0 0"/>
+    <child link="hokuyo"/>
+    <parent link="chassis"/>
+    <axis xyz="0 1 0" rpy="0 0 0"/>
+  </joint>
 </robot>

Commit message: 11.House your robot

File: project2/src/my_robot/urdf/my_robot.xacro (robot description, xacro)
@@ -1,4 +1,5 @@
 <?xml version='1.0'?>
 <robot name="my_robot" xmlns:xacro="http://www.ros.org/wiki/xacro">
+  <xacro:include filename="$(find my_robot)/urdf/my_robot.gazebo" />
   <link name="robot_footprint"></link>
   <joint name="robot_footprint_joint" type="fixed">
@@ -131,5 +132,7 @@
         <mesh filename="package://my_robot/meshes/hokuyo.dae"/>
       </geometry>
-      <material name="black"/>
+      <material name="black">
+        <color rgba="0 0 0 0"/>
+      </material>
     </visual>
     <collision name='hokuyo_collision'>
